File: kicad/coco9511pak.kicad_sch (KiCad schematic)
At the start: 36 parts, among them SW1 SW_DIP_x06, U1 74LS32, U10 74LS682, U11 74LS123, U12 74LS05, U13 74LS244, U14 74LS74, U15 PDME2-S5-S12-S, U16 Coco_Cart_Connector, U4 74LS04, U5 AM9511, U6 74LS374, U7 74LS00, U8 74LS30, U9 74LS08, X1 CXO_DIP14 4Mhz

Commit message: Update to v1.1
Parts:
- removed C15: .33uf, Capacitor_THT:C_Axial_L3.8mm_D2.6mm_P7.50mm_Horizontal, symbol Device:C
- removed U15: PDME2-S5-S12-S, Coco:PDME2-S5-S12-S, symbol Coco:PDME2-S5-S12-S
- removed unit 2 of U7
- added C16, C17: 22uF, Capacitor_THT:CP_Radial_D6.3mm_P2.50mm, symbol Device:C_Polarized
- added C3: .01uf, Capacitor_THT:C_Axial_L3.8mm_D2.6mm_P7.50mm_Horizontal, symbol Device:C
- added D1: 1N5818, Diode_THT:D_DO-41_SOD81_P10.16mm_Horizontal, symbol Diode:1N5818
- added JP2: Jumper_3_Open, Connector_PinHeader_2.54mm:PinHeader_1x03_P2.54mm_Vertical, symbol Jumper:Jumper_3_Open
- added L1: 22uH, Inductor_THT:L_Axial_L7.0mm_D3.3mm_P10.16mm_Horizontal_Fastron_MICC, symbol Device:L
- added R5: 215k, Resistor_THT:R_Axial_DIN0207_L6.3mm_D2.5mm_P7.62mm_Horizontal, symbol Device:R
- added R6: 24.9k, Resistor_THT:R_Axial_DIN0207_L6.3mm_D2.5mm_P7.62mm_Horizontal, symbol Device:R
- added R7: 5k, Resistor_THT:R_Axial_DIN0207_L6.3mm_D2.5mm_P7.62mm_Horizontal, symbol Device:R
- added U3: LT1373CN8, Package_DIP:DIP-8_W7.62mm, symbol Regulator_Switching:LT1373CN8
- C15: renamed from C16; value 100pf -> 47pf; footprint Resistor_THT:R_Axial_DIN0207_L6.3mm_D2.5mm_P7.62mm_Horizontal -> Capacitor_THT:C_Axial_L3.8mm_D2.6mm_P7.50mm_Horizontal
- R2: value 2.0k -> 3.3k
- U1, U12, U14, U4, U7, U8, U9, X1: footprint Package_DIP:DIP-14_W7.62mm_Socket -> Package_DIP:DIP-14_W7.62mm
- U10, U13, U6: footprint Package_DIP:DIP-20_W7.62mm_Socket -> Package_DIP:DIP-20_W7.62mm
- U11: footprint Package_DIP:DIP-16_W7.62mm_Socket -> Package_DIP:DIP-16_W7.62mm
- U5: footprint Package_DIP:DIP-24_W15.24mm_Socket -> Package_DIP:DIP-24_W15.24mm
Connections:
- net +5V is gone; now on net VCC: U10.20 (Vcc)
- net A0: now also U14.12 (D); no longer U5.21 (C/D*)
- net D5: now also U13.13 (I1b), U6.15 (O5); no longer U13.17 (I3b), U6.19 (O7)
- net D7: now also U13.17 (I3b), U6.19 (O7); no longer U13.13 (I1b), U6.15 (O5)
- net E: now also U10.17 (P7); no longer U1.1, U7.1, U9.12
- net GND: now also U1.12, U1.13, U12.7 (GND), U7.10, U7.9, U9.12, U9.13, C16.2, C17.2, R6.2, R7.2, U3.6 (GNDS), U3.7 (GND); no longer U10.17 (P7), U10.18 (Q7), U12.14 (VCC), U12.3, U14.11 (C), U14.12 (D), U14.3 (C), U4.13, U4.9
- net HALT*: now also JP1.2 (B); no longer JP1.1 (A)
- net LATCH_SELECT: now also U7.1; no longer U7.9
- net PROC_SELECT*: now also U1.2, U4.13; no longer U1.13
- net R*/W: now also U1.9; no longer U7.2
- net RD_LATCH*: now also U7.3; no longer U7.8
- net RD_PROC*: now also U9.1
- net RESET*: now also U14.1 (~{R}); no longer U9.1
- net R/W*: now also U1.1, U7.2; no longer U9.13
- net VCC: now also U10.18 (Q7), U12.14 (VCC), U3.4 (S/S); no longer C2.1, U12.7 (GND)
- net WR*: now also U1.3; no longer U1.11
- net CLK: now reaches U5.23 (CLK), X1.8 (OUT)
- net at U4.8: now also U12.3
- net +12V: now reaches U5.16 (VDD)
- net +12V: now also C2.1, JP2.2 (C)
- net at U9.11: no longer U7.10
- net C/D*: now reaches U14.9 (Q)
- net C/D*: now also U5.21 (C/D*)
- net at U12.4: now also JP1.1 (A), R4.1
- net at U9.3: now also U14.3 (C), U6.11 (Cp); no longer U14.1 (~{R})
- net at U4.12: now also U14.11 (C)
- net Cart12V: now reaches U16.2 (+12V)
- net Cart12V: now also JP2.1 (A)
- net Q: no longer names the net of U16.7 (Q)
- net Q: no longer U1.2
- new net: C17.1, D1.1 (K), JP2.3 (B), R5.1
- new net: R5.2, R6.1, U3.2 (FB)
- new net: C16.1, L1.1, U3.5 (Vin)
- new net: U4.9, U5.17 (PAUSE*), U9.2
- new net: D1.2 (A), L1.2, U3.8 (VSW)
- new net: C3.1, U3.1 (VC)
- new net: C3.2, R7.1
Other:
- moved on the sheet: C1, R4, U12B, U12G, U14B, U1B, U1D, U4D, U4E, U4F, U7C, U7D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

Commit message: Fixed missing vcc in boost circuit
Connections:
- net VCC: now also C16.1, L1.1, U3.5 (Vin)
Changed lines of the file:
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@@
+    (pin "1")
+  )
+  (symbol (lib_id "power:VCC") (at 285.75 58.42 0) (unit 1)
+    (in_bom yes) (on_board yes) (fields_autoplaced)
+    (property "Reference" "#PWR?" (id 0) (at 285.75 62.23 0)
+      (effects (font (size 1.27 1.27)) hide)
+    )
+    (property "Value" "VCC" (id 1) (at 285.75 53.34 0))
+    (property "Footprint" "" (id 2) (at 285.75 58.42 0)
+      (effects (font (size 1.27 1.27)) hide)
+    )
+    (property "Datasheet" "" (id 3) (at 285.75 58.42 0)
+      (effects (font (size 1.27 1.27)) hide)
+    )
     (pin "1")
   )
@@
       (reference "#PWR0113") (unit 1) (value "Gnd") (footprint "")
     )
+    (path "/0edca048-b9f6-44ca-83ea-9f9cd28f25c8"
+      (reference "#PWR?") (unit 1) (value "VCC") (footprint "")
+    )
     (path "/1ff809bd-80e3-46ff-b7e6-5fef8477146c"
